File: oscilliscope_board.kicad_pcb (KiCad board)
At the start: 4 copper layers, 98.5 x 97.5 mm, 40 parts, among them J1 Conn_Coaxial, J2 Conn_Coaxial, J3 Barrel_Jack, SW1 SW_Push, SW2 RotaryEncoder_Switch_MP, U2 ADC0832

Commit message: added mounting holes for stand-off legs
Parts:
- added H1: MountingHole_Pad, MountingHole:MountingHole_3.2mm_M3_DIN965_Pad, F.Cu at (82.8, 143.2)
- added H2: MountingHole_Pad, MountingHole:MountingHole_3.2mm_M3_DIN965_Pad, F.Cu at (82.8, 52.0)
- added H3: MountingHole_Pad, MountingHole:MountingHole_3.2mm_M3_DIN965_Pad, F.Cu at (175.0, 131.5)
- added H4: MountingHole_Pad, MountingHole:MountingHole_3.2mm_M3_DIN965_Pad, F.Cu at (165.0, 57.6)
Connections:
- net GNDA renamed GNDD
